File: Hardware/Revision2.0/SparrowCompass.kicad_pcb (KiCad board)
At the start: 4 copper layers, 72 x 94 mm, 82 parts, among them IC1 NEO-M8N-0, IC2 LSM303AGRTR, IC3 DRV8834RGER, IC4 XC6806A42011-G, IC5 TESEO-LIV3F, IC6 LSM9DS1TR, IC7 EE-SX1320, IC8 LDL1117S33R, IC9 LDL1117S33R, J1 Conn_01x04, J10 Conn_01x04, J2 Conn_Coaxial_Small, J3 USB4105-GF-A-060, J4 Conn_01x02, J5 Conn_01x02, J6 Conn_01x05, J7 Conn_01x10, J8 Conn_01x10, J9 Conn_01x10, U1 L3GD20, U2 TPD2EUSB30, U3 STM32F302CCTx, Y1 XRCGB25M000F3M00R0

Commit message: ENH: Hardware v2
Parts:
- removed C4, C5: 100n, Capacitor_SMD:C_0603_1608Metric
- removed D4: LED, LED_SMD:LED_0603_1608Metric
- removed IC3: DRV8834RGER, DRV8834RGER:QFN50P400X400X100-25N-D
- removed R10: 330R, Resistor_SMD:R_0603_1608Metric
- removed R7: 80R, Resistor_SMD:R_0603_1608Metric
- removed R8, R9: 200R, Resistor_SMD:R_0603_1608Metric
- added C33: 10u, Capacitor_Tantalum_SMD:CP_EIA-6032-15_Kemet-U, F.Cu at (160.0, 113.5)
- added C34: 10u, Capacitor_Tantalum_SMD:CP_EIA-6032-15_Kemet-U, F.Cu at (168.5, 113.5)
- added C35: 1u, Capacitor_Tantalum_SMD:CP_EIA-6032-15_Kemet-U, F.Cu at (137.2, 114.9)
- added C36: 100n, Capacitor_SMD:C_0603_1608Metric, F.Cu at (146.0, 112.1)
- added C37: 10u, Capacitor_Tantalum_SMD:CP_EIA-6032-15_Kemet-U, F.Cu at (166.0, 118.5)
- added C38: 1u, Capacitor_Tantalum_SMD:CP_EIA-6032-15_Kemet-U, F.Cu at (142.9, 105.4)
- added C39: 22u, Capacitor_Tantalum_SMD:CP_EIA-6032-15_Kemet-U, F.Cu at (159.0, 83.4)
- added C40: 2u2, Capacitor_SMD:C_0603_1608Metric, F.Cu at (161.5, 86.8)
- added C41: 100n, Capacitor_SMD:C_0603_1608Metric, F.Cu at (157.0, 90.9)
- added C42: 22n, Capacitor_SMD:C_0603_1608Metric, F.Cu at (163.0, 95.0)
- added C43: 10n, Capacitor_SMD:C_0603_1608Metric, F.Cu at (146.3, 61.9)
- added C44: 10u, Capacitor_Tantalum_SMD:CP_EIA-6032-15_Kemet-U, F.Cu at (136.0, 57.4)
- added C45: 100n, Capacitor_SMD:C_0603_1608Metric, F.Cu at (146.3, 60.3)
- added D8: LED, LED_SMD:LED_0603_1608Metric, F.Cu at (143.4, 123.7)
- added R27: 120R, Resistor_SMD:R_0603_1608Metric, F.Cu at (132.6, 109.0)
- added R28: 120R, Resistor_SMD:R_0603_1608Metric, F.Cu at (132.6, 110.7)
- added R29: 120R, Resistor_SMD:R_0603_1608Metric, F.Cu at (132.6, 112.4)
- added R30: 10k, Resistor_SMD:R_0603_1608Metric, F.Cu at (146.0, 108.8)
- added R31: 1k8, Resistor_SMD:R_0603_1608Metric, F.Cu at (145.9, 104.4)
- added R32: 1k, Resistor_SMD:R_0603_1608Metric, F.Cu at (148.3, 112.1)
- added R33: 1k, Resistor_SMD:R_0603_1608Metric, F.Cu at (149.9, 112.1)
- added R34: 10k, Resistor_SMD:R_0603_1608Metric, F.Cu at (130.5, 119.9)
- added R35: 1k, Resistor_SMD:R_0603_1608Metric, F.Cu at (153.0, 80.0)
- added R36: 820R, Resistor_SMD:R_0603_1608Metric, F.Cu at (157.0, 93.9)
- added R37: 130R, Resistor_SMD:R_0603_1608Metric, F.Cu at (166.0, 92.3)
- added R38: 130R, Resistor_SMD:R_0603_1608Metric, F.Cu at (166.0, 94.0)
- added R39: 1k, Resistor_SMD:R_0603_1608Metric, F.Cu at (161.5, 95.0)
- added R40: 47k, Resistor_SMD:R_0603_1608Metric, F.Cu at (160.0, 95.0)
- added R41: 10k, Resistor_SMD:R_0603_1608Metric, F.Cu at (140.1, 55.6)
- added R42: 10k, Resistor_SMD:R_0603_1608Metric, F.Cu at (140.9, 54.7)
- added R43: 10k, Resistor_SMD:R_0603_1608Metric, F.Cu at (144.0, 55.6)
- added R44: 10k, Resistor_SMD:R_0603_1608Metric, F.Cu at (143.2, 54.7)
- added R45: 10k, Resistor_SMD:R_0603_1608Metric, F.Cu at (139.6, 57.3)
- added R46: 10k, Resistor_SMD:R_0603_1608Metric, F.Cu at (139.6, 58.8)
- added R47: 10k, Resistor_SMD:R_0603_1608Metric, F.Cu at (168.8, 57.0)
- added R48: 10k, Resistor_SMD:R_0603_1608Metric, F.Cu at (168.8, 55.4)
- added R49: 0R0, Resistor_SMD:R_0603_1608Metric, F.Cu at (141.5, 66.2)
- added R50: 0R0, Resistor_SMD:R_0603_1608Metric, F.Cu at (143.2, 66.2)
- added R51: 0R0, Resistor_SMD:R_0603_1608Metric, F.Cu at (143.2, 64.7)
- added R52: 0R0, Resistor_SMD:R_0603_1608Metric, F.Cu at (141.5, 64.7)
- added R53: 0R0, Resistor_SMD:R_0603_1608Metric, F.Cu at (141.5, 63.2)
- added R54: 0R0, Resistor_SMD:R_0603_1608Metric, F.Cu at (143.2, 63.2)
- added S1: JS102011SAQN, JS102011SAQN:JS102011SAQN, F.Cu at (161.0, 126.0)
- added TP10: TestPoint, TestPoint:TestPoint_THTPad_D1.0mm_Drill0.5mm, F.Cu at (140.6, 126.5)
- added TP11: TestPoint, TestPoint:TestPoint_THTPad_D1.0mm_Drill0.5mm, F.Cu at (169.5, 121.4)
- added TP12: TestPoint, TestPoint:TestPoint_THTPad_D1.0mm_Drill0.5mm, F.Cu at (132.0, 115.3)
- added TP8: TestPoint, TestPoint:TestPoint_THTPad_D1.0mm_Drill0.5mm, F.Cu at (134.1, 115.3)
- added TP9: TestPoint, TestPoint:TestPoint_THTPad_D1.0mm_Drill0.5mm, F.Cu at (167.5, 121.4)
- added U4: STSPIN220, STSPIN220:VFQFPN-16_STM, F.Cu at (161.5, 90.5)
- C16: value 2u2 -> 220n
- C17: value 100n -> 220n
- J10: value Conn_01x04 -> Conn_01x05; footprint Connector_PinHeader_2.54mm:PinHeader_1x04_P2.54mm_Vertical -> Connector_PinHeader_2.54mm:PinHeader_1x05_P2.54mm_Vertical
- R14, R17: value 470R -> 130R
- R15, R18: value 10k -> 500m
- R16: value 10k -> 130R
- R23: value 470R -> 0R0
- moved J10 103.2 mm to (129.1, 115.8), turned to 180 degrees
- moved IC4 86.5 mm to (149.1, 108.0), turned to -90 degrees
- moved R26 80.9 mm to (137.5, 79.5), turned to -90 degrees
- moved R25 79.3 mm to (139.5, 79.5), turned to -90 degrees
- moved R21 77.7 mm to (141.5, 79.5), turned to -90 degrees
- moved D1 77.5 mm to (139.5, 75.0), turned to -90 degrees
- moved J9 74.2 mm to (135.5, 74.5), turned to -45 degrees
- moved IC6 72.3 mm to (142.9, 59.9), turned to -90 degrees
- moved IC8 66.0 mm to (160.0, 107.0), turned to 90 degrees
- moved IC5 64.2 mm to (161.3, 58.9), turned to 0 degrees
- moved IC9 54.2 mm to (168.5, 107.0), turned to 90 degrees
- moved D7 49.3 mm to (141.4, 123.7), turned to -90 degrees
- moved IC7 48.8 mm to (150.0, 80.0), turned to 90 degrees
- moved R14 44.8 mm to (147.0, 80.0), turned to 90 degrees
- moved C32 44.2 mm to (142.9, 113.1), turned to -90 degrees
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Connections:
- C16 pad 1: /1V75 -> +3.3V
- C17 pad 1: /1V75 -> +3.3V
- C17 pad 2: Net-(IC3-VCP) -> GND
- C28 pad 1: +3.3V -> Net-(IC6-C1)
- C7 pad 1: /1V75 -> Net-(IC9-VOUT_1)
- C8 pad 1: /1V75 -> Net-(IC9-VOUT_1)
- C9 pad 1: /1V75 -> Net-(IC9-VOUT_1)
- D7 pad 2: /1V75 -> /V_USB
- IC1 pad 11: Net-(IC1-RF_IN) -> /GPS_ANT
- IC4 pad 1: unconnected-(IC4-VIN-Pad1) -> /V_USB
- IC4 pad 10: unconnected-(IC4-OUT-Pad10) -> Net-(IC4-OUT)
- IC4 pad 2: unconnected-(IC4-ISET-Pad2) -> Net-(IC4-ISET)
- IC4 pad 3: unconnected-(IC4-THIN-Pad3) -> Net-(IC4-THIN)
- IC4 pad 4: unconnected-(IC4-VREG-Pad4) -> Net-(IC4-VREG)
- IC4 pad 5: unconnected-(IC4-PGB-Pad5) -> Net-(IC4-PGB)
- IC4 pad 6: unconnected-(IC4-CSO-Pad6) -> Net-(IC4-CSO)
- IC4 pad 7: unconnected-(IC4-VSS-Pad7) -> GND
- IC4 pad 8: unconnected-(IC4-SD-Pad8) -> GND
- IC4 pad 9: unconnected-(IC4-BAT-Pad9) -> Net-(IC4-BAT)
- IC5 pad 1: unconnected-(IC5-GND-Pad1) -> GND
- IC5 pad 10: unconnected-(IC5-GND_RF_1-Pad10) -> GND
- IC5 pad 11: unconnected-(IC5-RF_IN-Pad11) -> /GPS_ANT
- IC5 pad 12: unconnected-(IC5-GND_RF_2-Pad12) -> GND
- IC5 pad 16: unconnected-(IC5-SDA-Pad16) -> /I2C_SDA
- IC5 pad 17: unconnected-(IC5-SCL-Pad17) -> /I2C_SCL
- IC5 pad 5: unconnected-(IC5-WAKE-UP-Pad5) -> /GPS_INT
- IC5 pad 7: unconnected-(IC5-VCC_IO-Pad7) -> +3.3V
- IC5 pad 8: unconnected-(IC5-VCC-Pad8) -> +3.3V
- IC5 pad 9: unconnected-(IC5-SYS_RSTN-Pad9) -> /GPS_nReset
- IC6 pad 1: unconnected-(IC6-VDDIO_1-Pad1) -> +3.3V
- IC6 pad 10: unconnected-(IC6-INT_M-Pad10) -> /MAG_INT1
- IC6 pad 11: unconnected-(IC6-INT1_A/G-Pad11) -> /MAG_INT2
- IC6 pad 12: unconnected-(IC6-INT2_A/G-Pad12) -> /GYR_INT
- IC6 pad 13: unconnected-(IC6-DEN_A/G-Pad13) -> /GYR_DRDY
- IC6 pad 14: unconnected-(IC6-RES_1-Pad14) -> GND
- IC6 pad 15: unconnected-(IC6-RES_2-Pad15) -> GND
- IC6 pad 16: unconnected-(IC6-RES_3-Pad16) -> GND
- IC6 pad 17: unconnected-(IC6-RES_4-Pad17) -> GND
- IC6 pad 18: unconnected-(IC6-RES_5-Pad18) -> GND
- IC6 pad 19: unconnected-(IC6-GND_1-Pad19) -> GND
- IC6 pad 2: unconnected-(IC6-SCL/SPC-Pad2) -> /I2C_SCL
- IC6 pad 20: unconnected-(IC6-GND_2-Pad20) -> GND
- IC6 pad 21: unconnected-(IC6-CAP-Pad21) -> Net-(IC6-CAP)
- IC6 pad 22: unconnected-(IC6-VDD_1-Pad22) -> +3.3V
- IC6 pad 23: unconnected-(IC6-VDD_2-Pad23) -> +3.3V
- IC6 pad 24: unconnected-(IC6-C1-Pad24) -> Net-(IC6-C1)
- IC6 pad 3: unconnected-(IC6-VDDIO_2-Pad3) -> +3.3V
- IC6 pad 4: unconnected-(IC6-SDA/SDI/SDO-Pad4) -> /I2C_SDA
- IC6 pad 5: unconnected-(IC6-SDO_A/G-Pad5) -> Net-(IC6-SDO_A/G)
- IC6 pad 6: unconnected-(IC6-SDO_M-Pad6) -> Net-(IC6-SDO_M)
- IC6 pad 7: unconnected-(IC6-CS_A/G-Pad7) -> Net-(IC6-CS_A/G)
- IC6 pad 8: unconnected-(IC6-CS_M-Pad8) -> Net-(IC6-CS_M)
- IC6 pad 9: unconnected-(IC6-DRDY_M-Pad9) -> /MAG_DRDY
- IC7 pad 1: unconnected-(IC7-Pad1) -> Net-(IC7-Pad1)
- IC7 pad 2: unconnected-(IC7-Pad2) -> GND
- IC7 pad 3: unconnected-(IC7-Pad3) -> /MOT_SENSE
- IC7 pad 4: unconnected-(IC7-Pad4) -> +3.3V
- IC8 pad 1: unconnected-(IC8-GND-Pad1) -> GND
- IC8 pad 2: unconnected-(IC8-VOUT_1-Pad2) -> +3.3V
- IC8 pad 3: unconnected-(IC8-VIN-Pad3) -> /V_SYS
- IC8 pad 4: unconnected-(IC8-VOUT_2-Pad4) -> +3.3V
- IC9 pad 1: unconnected-(IC9-GND-Pad1) -> GND
- IC9 pad 2: unconnected-(IC9-VOUT_1-Pad2) -> Net-(IC9-VOUT_1)
- IC9 pad 3: unconnected-(IC9-VIN-Pad3) -> /V_SYS
- IC9 pad 4: unconnected-(IC9-VOUT_2-Pad4) -> Net-(IC9-VOUT_1)
- J10 pad 1: unconnected-(J10-Pin_1-Pad1) -> +3.3V
- J10 pad 2: unconnected-(J10-Pin_2-Pad2) -> Net-(J10-Pin_2)
- J10 pad 3: unconnected-(J10-Pin_3-Pad3) -> Net-(J10-Pin_3)
- J10 pad 4: unconnected-(J10-Pin_4-Pad4) -> Net-(J10-Pin_4)
- J2 pad 1: Net-(IC1-RF_IN) -> /GPS_ANT
- J3 pad SH3: GND -> unconnected-(J3-SHELL_GND__2-PadSH3)
- J3 pad SH4: GND -> unconnected-(J3-SHELL_GND__3-PadSH4)
- J4 pad 1: unconnected-(J4-Pin_1-Pad1) -> Net-(IC4-BAT)
- J5 pad 1: unconnected-(J5-Pin_1-Pad1) -> Net-(IC4-THIN)
- J7 pad 2: /MAG_DRDY -> /SENS_IO_1
- J7 pad 3: /MAG_INT1 -> /SENS_IO_2
- J7 pad 4: /GYR_DRDY -> /SENS_IO_3
- J8 pad 2: /MAG_DRDY -> /SENS_IO_1
- J8 pad 3: /MAG_INT1 -> /SENS_IO_2
- J8 pad 4: /GYR_DRDY -> /SENS_IO_3
- J9 pad 1: unconnected-(J9-Pin_1-Pad1) -> +3.3V
- J9 pad 10: unconnected-(J9-Pin_10-Pad10) -> GND
- J9 pad 2: unconnected-(J9-Pin_2-Pad2) -> +3.3V
- J9 pad 3: unconnected-(J9-Pin_3-Pad3) -> /IO_1
- J9 pad 4: unconnected-(J9-Pin_4-Pad4) -> /IO_2
- J9 pad 5: unconnected-(J9-Pin_5-Pad5) -> /IO_3
- J9 pad 6: unconnected-(J9-Pin_6-Pad6) -> /IO_4
- J9 pad 7: unconnected-(J9-Pin_7-Pad7) -> /IO_5
- J9 pad 8: unconnected-(J9-Pin_8-Pad8) -> /IO_6
- J9 pad 9: unconnected-(J9-Pin_9-Pad9) -> GND
- R14 pad 1: unconnected-(R14-Pad1) -> Net-(IC7-Pad1)
- R15 pad 1: +3.3V -> Net-(U4-SENSEA)
- R15 pad 2: Net-(IC3-CONFIG) -> GND
- R17 pad 1: Net-(IC3-NFAULT) -> +3.3V
- R18 pad 1: +3.3V -> Net-(U4-SENSEB)
- R18 pad 2: Net-(IC3-M1) -> GND
- R19 pad 1: +3.3V -> Net-(U4-REF)
- R19 pad 2: Net-(IC3-M0_/_APHASE) -> +3.3V
- R23 pad 1: GND -> Net-(IC9-VOUT_1)
- R23 pad 2: Net-(D7-K) -> +3.3V
- TP4 pad 1: /1V75 -> Net-(IC9-VOUT_1)
- U3 pad 12: /MAG_DRDY -> /SENS_IO_1
- U3 pad 13: /MAG_INT1 -> /SENS_IO_2
- U3 pad 14: /GYR_DRDY -> /SENS_IO_3
- U3 pad 18: unconnected-(U3-PB0-Pad18) -> /IO_1
- U3 pad 19: unconnected-(U3-PB1-Pad19) -> /IO_2
- U3 pad 20: unconnected-(U3-PB2-Pad20) -> /IO_3
- U3 pad 21: unconnected-(U3-PB10-Pad21) -> /MOT_STBY
- U3 pad 22: /MOT_nEnable -> /MOT_Enable
- U3 pad 27: /MOT_SENS_B -> /MOT_SENSE
- U3 pad 28: /MOT_SENS_A -> unconnected-(U3-PB15-Pad28)
- U3 pad 29: unconnected-(U3-PA8-Pad29) -> /RFID_EN
- U3 pad 30: unconnected-(U3-PA9-Pad30) -> /USART_TX
- U3 pad 31: unconnected-(U3-PA10-Pad31) -> /USART_RX
- U3 pad 39: unconnected-(U3-PB3-Pad39) -> /IO_4
- U3 pad 40: unconnected-(U3-PB4-Pad40) -> /IO_5
- U3 pad 41: unconnected-(U3-PB5-Pad41) -> /IO_6
Routing:
- net /GYR_DRDY: track 88.2 -> 4.75 mm, vias 2 -> 0
- net /MAG_INT1: track 99.2 -> 24.1 mm, vias 1 -> 3
- net /MAG_DRDY: track 93.0 -> 19.3 mm, vias 1 -> 3
- net /V_BAT: track 63.6 -> 0.00 mm
- net GND: track 69.8 -> 129.2 mm, vias 66 -> 199
- net /MOT_nEnable: track 58.4 -> 0.00 mm, vias 2 -> 0
- net /1V75: track 44.8 -> 0.00 mm
- net /GPS_nReset: track 95.3 -> 53.0 mm, vias 1 -> 2
- net /SENS_IO_3: track 0.00 -> 42.2 mm, vias 0 -> 1
- net /V_SYS: track 0.00 -> 40.2 mm, vias 0 -> 6
- net /SENS_IO_1: track 0.00 -> 38.6 mm, vias 0 -> 1
- net /SENS_IO_2: track 0.00 -> 38.6 mm, vias 0 -> 1
- net /GPS_INT: track 97.6 -> 59.4 mm
- net /MOT_SENSE: track 0.00 -> 35.5 mm, vias 0 -> 2
- net /MOT_STBY: track 0.00 -> 33.0 mm, vias 0 -> 2
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- added copper zone on In2.Cu, net +3.3V
- added copper zone on In2.Cu, net /V_SYS
- added copper zone on In1.Cu, net GND
- removed copper zone on In1.Cu, net +3.3V
- removed copper zone on In2.Cu, net GND
Other:
- board size 72 x 94 mm -> 56 x 75 mm
- board text added: "-BAT+"
- board text added: "1"
- board text added: "2"
- board text added: "3"
- board text added: "3v3"
- board text added: "4"
- board text added: "5"
- board text added: "6"
- board text added: "A B"
- board text added: "BAT"
- board text added: "CHG"
- board text added: "CLK"
- board text added: "EN"
- board text added: "GND"
- board text added: "GPS_I"
- board text added: "GPS_R"
- board text added: "I2C_C"
- board text added: "I2C_D"
- board text added: "IO"
- board text added: "PWR"
- board text added: "RST"
- board text added: "RX"
- board text added: "SIO1"
- board text added: "SIO2"
- board text added: "SIO3"
- board text added: "SYS"
- board text added: "UART"
- board text added: "USB"
- board text removed: "- BAT +"
- board text removed: "1v75"
- board text removed: "3V3"
- board text removed: "C"
- board text removed: "D"
- board text removed: "FAULT"
- board text removed: "G"
- board text removed: "S1"
- board text removed: "S2"
- board text removed: "V"
- board text removed: "VBat"
