File: Hardware/Revision2.0/SparrowCompass.kicad_sch (KiCad schematic)
At the start: 77 parts, among them IC1 NEO-M8N-0, IC2 LSM303AGRTR, IC3 DRV8834RGER, IC4 XC6806A42011-G, IC5 TESEO-LIV3F, IC6 LSM9DS1TR, IC7 EE-SX1320, IC8 LDL1117S33R, IC9 LDL1117S33R, J1 Conn_01x04, J10 Conn_01x04, J2 Conn_Coaxial_Small, J3 USB4105-GF-A-060, J4 Conn_01x02, J5 Conn_01x02, J6 Conn_01x05, J7 Conn_01x10, J8 Conn_01x10, J9 Conn_01x10, U1 L3GD20, U2 TPD2EUSB30, U3 STM32F302CCTx, Y1 XRCGB25M000F3M00R0

Commit message: ENH: Hardware v2
Parts:
- removed D4: LED, LED_SMD:LED_0603_1608Metric, symbol Device:LED
- removed IC3: DRV8834RGER, DRV8834RGER:QFN50P400X400X100-25N-D, symbol DRV8834RGER:DRV8834RGER
- removed J10: Conn_01x04, Connector_PinHeader_2.54mm:PinHeader_1x04_P2.54mm_Vertical, symbol Connector_Generic:Conn_01x04
- added C35, C38: 1u, Capacitor_Tantalum_SMD:CP_EIA-6032-15_Kemet-U, symbol Device:C_Polarized
- added C36, C41, C45: 100n, Capacitor_SMD:C_0603_1608Metric, symbol Device:C
- added C37, C44: 10u, Capacitor_Tantalum_SMD:CP_EIA-6032-15_Kemet-U, symbol Device:C_Polarized
- added C39: 22u, Capacitor_Tantalum_SMD:CP_EIA-6032-15_Kemet-U, symbol Device:C_Polarized
- added C40: 2u2, Capacitor_SMD:C_0603_1608Metric, symbol Device:C
- added C42: 22n, Capacitor_SMD:C_0603_1608Metric, symbol Device:C
- added C43: 10n, Capacitor_SMD:C_0603_1608Metric, symbol Device:C
- added D7, D8: LED, LED_SMD:LED_0603_1608Metric, symbol Device:LED
- added J10: Conn_01x05, Connector_PinHeader_2.54mm:PinHeader_1x05_P2.54mm_Vertical, symbol Connector_Generic:Conn_01x05
- added R27, R28, R29: 120R, Resistor_SMD:R_0603_1608Metric, symbol Device:R
- added R30, R34, R41, R42, R43, R44, R45, R46, R47, R48: 10k, Resistor_SMD:R_0603_1608Metric, symbol Device:R
- added R31: 1k8, Resistor_SMD:R_0603_1608Metric, symbol Device:R
- added R32, R33, R35, R39: 1k, Resistor_SMD:R_0603_1608Metric, symbol Device:R
- added R36: 820R, Resistor_SMD:R_0603_1608Metric, symbol Device:R
- added R37, R38: 130R, Resistor_SMD:R_0603_1608Metric, symbol Device:R
- added R40: 47k, Resistor_SMD:R_0603_1608Metric, symbol Device:R
- added R49, R50, R51, R52, R53, R54: 0R0, Resistor_SMD:R_0603_1608Metric, symbol Device:R
- added S1: JS102011SAQN, JS102011SAQN:JS102011SAQN, symbol JS102011SAQN:JS102011SAQN
- added TP10, TP11, TP12, TP8, TP9: TestPoint, TestPoint:TestPoint_THTPad_D1.0mm_Drill0.5mm, symbol Connector:TestPoint
- added U4: STSPIN220, STSPIN220:VFQFPN-16_STM, symbol STSPIN220:STSPIN220
- C16: value 2u2 -> 220n
- C17: value 100n -> 220n
- IC4: footprint XC6806A42011G -> XC6806A42011-G:XC6806A42011G
- IC5: footprint SON110P970X1010X230-18N -> TESO-LIV3F:SON110P970X1010X230-18N
- IC6: footprint LGA-24L(3X3.5X1MM) -> LSM9DS1TR:LGA-24L_3X3.5X1MM_
- IC7: footprint EE-SX1320 -> EE-SX1320:EE-SX1320
- IC8, IC9: footprint SOT230P700X180-4N -> LDL1117S33R:SOT230P700X180-4N
- R14, R17: value 470R -> 130R
- R15, R18: value 10k -> 500m
- R16: value 10k -> 130R
Connections:
- net 1V75 is gone; now on net +3.3V: C16.1, C17.1
- net MOT_SENS_B is gone; now on net MOT_SENSE: U3.27 (PB14)
- net +3.3V: now also IC5.7 (VCC_IO), IC5.8 (VCC), IC6.1 (VDDIO_1), IC6.22 (VDD_1), IC6.23 (VDD_2), IC6.3 (VDDIO_2), IC7.4, J9.1 (Pin_1), J9.2 (Pin_2), R17.1, R19.2, C44.1, C45.1, J10.1 (Pin_1), R41.1, R43.1, R45.1, R46.1, R47.1, R48.1; no longer C28.1, R15.1, R18.1, R19.1
- net GND: now also C17.2, IC4.7 (VSS), IC4.8 (SD), IC5.1 (GND), IC5.10 (GND_RF_1), IC5.12 (GND_RF_2), IC6.14 (RES_1), IC6.15 (RES_2), IC6.16 (RES_3), IC6.17 (RES_4), IC6.18 (RES_5), IC6.19 (GND_1), IC6.20 (GND_2), IC7.2, J9.10 (Pin_10), J9.9 (Pin_9), R15.2, R18.2, C35.2, C36.2, C37.2, C38.2, C39.2, C40.2, C41.1, C42.1, C43.2, C44.2, C45.2, J10.5 (Pin_5), R31.1, R34.2, R35.2, R36.1, R37.2, R38.2, R40.2, R42.2, R44.2, TP11.1, TP12.1, U4.17 (EPAD), U4.7 (GND); no longer J3.SH3 (SHELL_GND__2), J3.SH4 (SHELL_GND__3)
- net GPS_INT: now also IC5.5 (WAKE-UP)
- net GPS_nReset: now also IC5.9 (SYS_RSTN)
- net GYR_DRDY: now also IC6.13 (DEN_A/G), R53.2; no longer J7.4 (Pin_4), J8.4 (Pin_4), U3.14 (PA4)
- net GYR_INT: now also IC6.12 (INT2_A/G), R54.1
- net I2C_SCL: now also IC5.17 (SCL), IC6.2 (SCL/SPC), R48.2
- net I2C_SDA: now also IC5.16 (SDA), IC6.4 (SDA/SDI/SDO), R47.2
- net MAG_DRDY: now also IC6.9 (DRDY_M), R49.2, R52.1; no longer J7.2 (Pin_2), J8.2 (Pin_2), U3.12 (PA2)
- net MAG_INT1: now also IC6.10 (INT_M), R50.1; no longer J7.3 (Pin_3), J8.3 (Pin_3), U3.13 (PA3)
- net MAG_INT2: now also IC6.11 (INT1_A/G), R51.2
- net MOT_A1: now also U4.3 (OUTA1)
- net MOT_A2: now also U4.5 (OUTA2)
- net MOT_B1: now also U4.10 (OUTB1)
- net MOT_B2: now also U4.8 (OUTB2)
- net MOT_DIR: now also U4.1 (DIR/MODE4)
- net MOT_STEP: now also U4.2 (STCK/MODE3)
- net V_USB: now also IC4.1 (VIN), C38.1, D7.2 (A), D8.2 (A), TP10.1
- net GPS_ANT: now reaches IC5.11 (RF_IN)
- net GPS_ANT: now also IC1.11 (RF_IN), J2.1 (In)
- net IO_1: now reaches J9.3 (Pin_3)
- net IO_1: now also U3.18 (PB0)
- net IO_2: now reaches J9.4 (Pin_4)
- net IO_2: now also U3.19 (PB1)
- net IO_3: now reaches J9.5 (Pin_5)
- net IO_3: now also U3.20 (PB2)
- net IO_4: now reaches J9.6 (Pin_6)
- net IO_4: now also U3.39 (PB3)
- net IO_5: now reaches J9.7 (Pin_7)
- net IO_5: now also U3.40 (PB4)
- net IO_6: now reaches J9.8 (Pin_8)
- net IO_6: now also U3.41 (PB5)
- net at IC4.10 (OUT): now also S1.2 (COM)
- net at IC4.2 (ISET): now also R31.2
- net at IC4.3 (THIN): now also J5.1 (Pin_1), R30.2, R34.1
- net at IC4.4 (VREG): now also C36.1, R30.1
- net at IC4.5 (PGB): now also R32.2
- net at IC4.6 (CSO): now also R33.1
- net at IC4.9 (BAT), J4.1 (Pin_1): now also C35.1, TP8.1
- net at IC7.1: now also R14.1
- net MOT_SENSE: now reaches IC7.3
- net MOT_SENSE: now also R35.1
- net at R17.2: now also R38.1, U4.15 (MODE2)
- net at R16.2: now also R37.1, U4.16 (MODE1)
- net MOT_STBY: now reaches U3.21 (PB10)
- net MOT_STBY: now also U4.14 (STBY/RESET)
- net RFID_EN: now reaches U3.29 (PA8)
- net RFID_EN: now also R27.1
- net USART_TX: now reaches U3.30 (PA9)
- net USART_TX: now also R28.1
- net USART_RX: now reaches U3.31 (PA10)
- net USART_RX: now also R29.1
- net at IC6.21 (CAP): now also C43.1
- net at IC6.24 (C1): now also C28.1
- net at IC6.5 (SDO_A/G): now also R43.2, R44.1
- net at IC6.6 (SDO_M): now also R41.2, R42.1
- net at IC6.7 (CS_A/G): now also R45.2
- net at IC6.8 (CS_M): now also R46.2
- net MOT_SENS_A: no longer names the net of U3.28 (PB15)
- net MOT_nEnable renamed MOT_Enable
- net MOT_Enable: now also U4.13 (EN/FAULT)
- net V_BAT renamed V_SYS
- net V_SYS: now also C37.1, C39.1, C40.1, S1.3 (N.O.), TP9.1, U4.6 (VS)
- new net: D7.1 (K), R32.1
- new net: J10.2 (Pin_2), R29.2
- new net: J10.3 (Pin_3), R28.2
- new net: J10.4 (Pin_4), R27.2
- new net: R39.1, R40.1, U4.12 (TOFF)
- new net: C42.2, R39.2
- new net: C41.2, R19.1, R36.2, U4.11 (REF)
- new net: D8.1 (K), R33.2
- new net: R18.1, U4.9 (SENSEB)
- new net: R15.1, U4.4 (SENSEA)
- new net SENS_IO_1: J7.2 (Pin_2), J8.2 (Pin_2), R49.1, R50.2, U3.12 (PA2)
- new net SENS_IO_2: J7.3 (Pin_3), J8.3 (Pin_3), R51.1, R52.2, U3.13 (PA3)
- new net SENS_IO_3: J7.4 (Pin_4), J8.4 (Pin_4), R53.1, R54.2, U3.14 (PA4)
- no-connect marks 17 -> 27
Other:
- note added: "Accelerometer / Gyroscope"
- note added: "Battery Charger"
- note added: "Charging"
- note added: "GPS"
- note added: "GPS Alternative"
- note added: "Magnetometer"
- note added: "Optical Sensor"
- note added: "Orientation Alternative"
- note added: "Power Good"
- note removed: "Power"
- moved on the sheet: C10, C11, C12, C13, C14, C15, C18, C19, C20, C21, C22, C23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
